File: rp2040_trackball_mouse.kicad_pcb (KiCad board)
At the start: 2 copper layers, 92 x 57 mm, 29 parts, among them J1 Conn_01x05, J2 Conn_01x06, J5 Conn_02x08_Odd_Even, J6 Conn_02x08_Odd_Even, SW1 SW_Push, SW2 SW_Push, SW3 SW_Push, SW4 SW_Push, U1 NJM4580, U2 PT5529B/L2/H3

Commit message: ホイールがぎこちないのを記述
Parts:
- U1: value NJM4580 -> LMV393D
Changed lines of the file:
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@@
   (net 12 "L_BTN")
   (net 13 "Net-(R13-Pad1)")
-  (net 14 "Net-(R23-Pad2)")
+  (net 14 "Net-(R14-Pad1)")
   (net 15 "Net-(R17-Pad1)")
   (net 16 "Net-(R19-Pad1)")
@@
     (fp_line (start 0.8 -0.4125) (end -0.8 -0.4125) (layer "B.Fab") (width 0.1))
     (pad "1" smd roundrect locked (at -0.9125 0 180) (size 0.975 0.95) (layers "B.Cu" "B.Paste" "B.Mask") (roundrect_rratio 0.25)
-      (net 14 "Net-(R23-Pad2)") (pintype "passive"))
+      (net 14 "Net-(R14-Pad1)") (pintype "passive"))
     (pad "2" smd roundrect locked (at 0.9125 0 180) (size 0.975 0.95) (layers "B.Cu" "B.Paste" "B.Mask") (roundrect_rratio 0.25)
       (net 24 "VBUS") (pintype "passive"))
@@
       (net 3 "Net-(C10-Pad2)") (pintype "passive"))
     (pad "2" smd roundrect locked (at 0.9125 0) (size 0.975 0.95) (layers "B.Cu" "B.Paste" "B.Mask") (roundrect_rratio 0.25)
-      (net 14 "Net-(R23-Pad2)") (pintype "passive"))
+      (net 14 "Net-(R14-Pad1)") (pintype "passive"))
     (model "${KISYS3DMOD}/Resistor_SMD.3dshapes/R_0603_1608Metric.wrl"
       (offset (xyz 0 0 0))
@@
       (effects (font (size 1 1) (thickness 0.15)) (justify mirror))
     )
-    (fp_text value "NJM4580" (at 0 -3.4) (layer "B.Fab")
+    (fp_text value "LMV393D" (at 0 -3.4) (layer "B.Fab")
       (effects (font (size 1 1) (thickness 0.15)) (justify mirror))
     )
@@
     (fp_line (start -1.95 1.475) (end -0.975 2.45) (layer "B.Fab") (width 0.1))
     (pad "1" smd roundrect locked (at -2.625 1.905 180) (size 1.65 0.6) (layers "B.Cu" "B.Paste" "B.Mask") (roundrect_rratio 0.25)
-      (net 14 "Net-(R23-Pad2)") (pintype "output"))
+      (net 14 "Net-(R14-Pad1)") (pintype "output"))
     (pad "2" smd roundrect locked (at -2.625 0.635 180) (size 1.65 0.6) (layers "B.Cu" "B.Paste" "B.Mask") (roundrect_rratio 0.25)
       (net 13 "Net-(R13-Pad1)") (pinfunction "-") (pintype "input"))

Commit message: 仮に入れていた値を削除
Parts:
- C10, C11: value 0.1u(not Mount) -> (not Mount)
Changed lines of the file:
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@@
       (effects (font (size 1 1) (thickness 0.15)) (justify mirror))
     )
-    (fp_text value "0.1u(not Mount)" (at 3.429 0) (layer "B.Fab")
+    (fp_text value "(not Mount)" (at 3.429 0) (layer "B.Fab")
       (effects (font (size 1 1) (thickness 0.15)) (justify mirror))
     )
@@
       (effects (font (size 1 1) (thickness 0.15)) (justify mirror))
     )
-    (fp_text value "0.1u(not Mount)" (at -3.175 0) (layer "B.Fab")
+    (fp_text value "(not Mount)" (at -3.175 0) (layer "B.Fab")
       (effects (font (size 1 1) (thickness 0.15)) (justify mirror))
     )
